File: catEars.kicad_pcb (KiCad board)
At the start: 2 copper layers, 41.3 x 41.4 mm, 31 parts, among them J1 Conn_01x03_Socket, J2 Conn_01x03_Socket, U1 ESP-01v090, U1_ PinSocket_2x04_P2.54mm_Vertic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, U2 AMS1117-3.3

Commit message: changed C11 value
Parts:
- C11: value 220uF -> 22uF
